File: GeneralRecruitmentFlyer.kicad_pcb (KiCad board)
At the start: 2 copper layers, 59.7 x 95.5 mm, 188 parts, among them SW1 3P1T_Fused, U1 VNH5019A-E, U10 LS_4, U2 VNH5019A-E, U3 3.3V_OKI, U4 LS_1, U5 LS_2, U6 TM4C129E_Launchpad_X9, U7 Picoblade-3, U8 Picoblade-3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

Commit message: Fixed Van's email
Other:
- board text added: "Joining the Team or Have Questions? Contact Marsrover@mst.edu, Jacob Lipina (jrlwd5@mst.edu), or Andrew Van Horn (asvdgv@mst.edu)"
- board text removed: "Joining the Team or Have Questions? Contact Marsrover@mst.edu, Jacob Lipina (jrlwd5@mst.edu), or Andrew Van Horn (asvgdv@mst.edu)"
Changed lines of the file:
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@@
     (links 259)
     (no_connects 0)
-    (area 116.32154 81.433999 192.4064 234.209661)
+    (area 117.958399 138.481599 177.748401 234.034801)
     (thickness 1.6)
     (drawings 63)
@@
     (effects (font (size 5 2.5) (thickness 0.3)))
   )
-  (gr_text "Joining the Team or Have Questions? Contact Marsrover@mst.edu, \nJacob Lipina (jrlwd5@mst.edu), or Andrew Van Horn (asvgdv@mst.edu)" (at 148.082 231.394) (layer F.SilkS)
+  (gr_text "Joining the Team or Have Questions? Contact Marsrover@mst.edu, \nJacob Lipina (jrlwd5@mst.edu), or Andrew Van Horn (asvdgv@mst.edu)" (at 148.082 231.394) (layer F.SilkS)
     (effects (font (size 1.1 1.05) (thickness 0.25)))
   )
