File: ShimbleBoard_Hardware/ShimbleBoard_Hardware.kicad_pcb (KiCad board)
At the start: 2 copper layers, 61 x 91.6 mm, 39 parts, among them U1 TM4C129E_Launchpad, U2 OKI, U3 OKI

Commit message: Updates
Parts:
- added G***: LOGO, MRDT_Silkscreens:0_MRDT_Logo_20mm, F.Cu at (106.9, 134.4)
- moved G*** 2.16 mm to (123.4, 116.6)
Other:
- board text added: "#ROVESOHARD"
- board text added: "Become a Martian & Join Today!!!"
- board text added: "Curiosity and Opprotunity Awaits. Want to Join or have Question? Contact Marsrover@mst.edu"
- board text added: "MARS ROVER DESIGN TEAM"
- board text added: "Today. Tomorrow. Forever."
- board text removed: "ROVE SO HARD"
